File: hardware/pcb/F407_mini/F407_mini.kicad_pcb (KiCad board)
At the start: 2 copper layers, 63.5 x 91.4 mm, 37 parts, among them J1 Conn_01x03, J10 Conn_01x03, J11 Conn_01x03, J12 Conn_01x03, J13 Conn_01x03, J14 Conn_01x03, J15 Conn_01x03, J16 Conn_01x03, J17 Conn_01x03, J18 Conn_01x03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

Commit message: flip connectors
Parts:
- J19, J20, J21: moved to F.Cu
- moved J20 2.54 mm to (157.5, 147.3), turned to 180 degrees
- moved J21 2.54 mm to (154.9, 106.7), turned to 270 degrees
- moved J19 2.54 mm to (127.0, 147.3), turned to 180 degrees
Connections:
- J19 pad 10: Net-(J19-Pad10) -> /B7
- J19 pad 11: /B5 -> Net-(J19-Pad11)
- J19 pad 12: Net-(J19-Pad12) -> /B5
- J19 pad 23: Net-(J19-Pad23) -> /C11
- J19 pad 24: /C11 -> Net-(J19-Pad24)
- J19 pad 25: Net-(J19-Pad25) -> /A15
- J19 pad 26: /A15 -> Net-(J19-Pad26)
- J19 pad 35: /C6 -> Net-(J19-Pad35)
- J19 pad 36: Net-(J19-Pad36) -> /C6
- J19 pad 7: Net-(J19-Pad7) -> /B8
- J19 pad 8: /B8 -> Net-(J19-Pad8)
- J19 pad 9: /B7 -> Net-(J19-Pad9)
- J20 pad 11: Net-(J20-Pad11) -> /E5
- J20 pad 12: /E5 -> Net-(J20-Pad12)
- J20 pad 13: /E6 -> Net-(J20-Pad13)
- J20 pad 14: Net-(J20-Pad14) -> /E6
- J20 pad 21: /A0 -> /A2
- J20 pad 22: /A2 -> /A0
- J20 pad 23: /A1 -> /A3
- J20 pad 24: /A3 -> /A1
- J20 pad 31: /B0 -> /B1
- J20 pad 32: /B1 -> /B0
- J20 pad 35: Net-(J20-Pad35) -> /E9
- J20 pad 36: /E9 -> Net-(J20-Pad36)
- J21 pad 1: /E11 -> Net-(J21-Pad1)
- J21 pad 11: /B15 -> /B14
- J21 pad 12: /B14 -> /B15
- J21 pad 2: Net-(J21-Pad2) -> /E11
- J21 pad 3: /E13 -> Net-(J21-Pad3)
- J21 pad 4: Net-(J21-Pad4) -> /E13
- J21 pad 5: Net-(J21-Pad5) -> /E14
- J21 pad 6: /E14 -> Net-(J21-Pad6)
- J21 pad 7: /B11 -> /B10
- J21 pad 8: /B10 -> /B11

Commit message: F407 mini board RC0
Parts:
- moved J23 1.27 mm to (116.8, 87.6)
- moved C2 1.27 mm to (132.1, 95.2)
- moved C4 1.27 mm to (160.0, 95.2)
- moved J22 1.27 mm to (146.1, 95.2)
- moved J24 1.27 mm to (116.8, 82.5)
- moved J25 1.27 mm to (116.8, 77.5)
- moved J26 1.27 mm to (116.8, 72.4)
Other:
- board size 63.5 x 91.4 mm -> 63.5 x 92.7 mm
Changed lines of the file:
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@@
-(kicad_pcb (version 20171130) (host pcbnew "(5.1.4)-1")
+(kicad_pcb (version 20171130) (host pcbnew "(5.1.5)-3")
   (general
     (thickness 1.6)
-    (drawings 5)
+    (drawings 9)
     (tracks 110)
     (zones 0)
@@
     (32 B.Adhes user hide)
     (33 F.Adhes user hide)
-    (34 B.Paste user hide)
+    (34 B.Paste user)
     (35 F.Paste user hide)
     (36 B.SilkS user)
@@
     (38 B.Mask user hide)
     (39 F.Mask user hide)
-    (40 Dwgs.User user hide)
+    (40 Dwgs.User user)
     (41 Cmts.User user hide)
     (42 Eco1.User user hide)
@@
     (solder_mask_min_width 0.25)
     (aux_axis_origin 0 0)
-    (visible_elements 7FFFFFFF)
+    (visible_elements 7FFFFF7F)
     (pcbplotparams
       (layerselection 0x010fc_ffffffff)
       (usegerberextensions false)
-      (usegerberattributes false)
+      (usegerberattributes true)
       (usegerberadvancedattributes false)
       (creategerberjobfile false)
-      (excludeedgelayer true)
+      (excludeedgelayer false)
       (linewidth 0.100000)
       (plotframeref false)
@@
       (outputformat 1)
       (mirror false)
-      (drillshape 1)
+      (drillshape 0)
       (scaleselection 1)
-      (outputdirectory ""))
+      (outputdirectory "gerber/"))
   )
   (net 0 "")
@@
     (descr "Through hole straight pin header, 1x03, 2.54mm pitch, single row")
     (tags "Through hole pin header THT 1x03 2.54mm single row")
-    (fp_text reference J28 (at 0 -2.33 90) (layer F.SilkS)
+    (fp_text reference J28 (at 0 -2.33 90) (layer F.SilkS) hide
       (effects (font (size 1 1) (thickness 0.15)))
     )
@@
     (descr "Through hole straight pin header, 1x03, 2.54mm pitch, single row")
     (tags "Through hole pin header THT 1x03 2.54mm single row")
-    (fp_text reference J27 (at 0 -2.33 90) (layer F.SilkS)
+    (fp_text reference J27 (at 0 -2.33 90) (layer F.SilkS) hide
       (effects (font (size 1 1) (thickness 0.15)))
     )
@@
   )
   (module Connector_PinHeader_2.54mm:PinHeader_2x22_P2.54mm_Vertical (layer F.Cu)
-    (at 116.84 73.66 90)
+    (at 116.84 72.39 90)
     (descr "Through hole straight pin header, 2x22, 2.54mm pitch, double rows")
     (tags "Through hole pin header THT 2x22 2.54mm double row")
@@
   )
   (module Connector_PinHeader_2.54mm:PinHeader_2x22_P2.54mm_Vertical (layer F.Cu)
-    (at 116.84 78.74 90)
+    (at 116.84 77.47 90)
     (descr "Through hole straight pin header, 2x22, 2.54mm pitch, double rows")
     (tags "Through hole pin header THT 2x22 2.54mm double row")
@@
   )
   (module Connector_PinHeader_2.54mm:PinHeader_2x22_P2.54mm_Vertical (layer F.Cu)
-    (at 116.84 83.82 90)
+    (at 116.84 82.55 90)
     (descr "Through hole straight pin header, 2x22, 2.54mm pitch, double rows")
     (tags "Through hole pin header THT 2x22 2.54mm double row")
@@
   )
   (module Connector_PinHeader_2.54mm:PinHeader_2x22_P2.54mm_Vertical (layer F.Cu)
-    (at 116.84 88.9 90)
+    (at 116.84 87.63 90)
     (descr "Through hole straight pin header, 2x22, 2.54mm pitch, double rows")
     (tags "Through hole pin header THT 2x22 2.54mm double row")
@@
   )
   (module Connector_PinHeader_2.54mm:PinHeader_1x03_P2.54mm_Vertical (layer F.Cu)
-    (at 146.05 96.52 270)
+    (at 146.05 95.25 270)
     (descr "Through hole straight pin header, 1x03, 2.54mm pitch, single row")
     (tags "Through hole pin header THT 1x03 2.54mm single row")
@@
   )
   (module Capacitor_THT:CP_Radial_D10.0mm_P5.00mm (layer F.Cu)
-    (at 160.02 96.52 180)
+    (at 160.02 95.25 180)
     (descr "CP, Radial series, Radial, pin pitch=5.00mm, , diameter=10mm, Electrolytic Capacitor")
     (tags "CP Radial series Radial pin pitch 5.00mm  diameter 10mm Electrolytic Capacitor")
@@
   )
   (module Capacitor_THT:CP_Radial_D10.0mm_P5.00mm (layer F.Cu)
-    (at 132.08 96.52 180)
+    (at 132.08 95.25 180)
     (descr "CP, Radial series, Radial, pin pitch=5.00mm, , diameter=10mm, Electrolytic Capacitor")
     (tags "CP Radial series Radial pin pitch 5.00mm  diameter 10mm Electrolytic Capacitor")
@@
     (pad 1 thru_hole circle (at 0 0) (size 6.4 6.4) (drill 3.2) (layers *.Cu *.Mask))
   )
+  (dimension 53.34 (width 0.15) (layer Dwgs.User)
+    (gr_text "53.340 mm" (at 143.51 166.399999) (layer Dwgs.User)
+      (effects (font (size 1 1) (thickness 0.15)))
+    )
+    (feature1 (pts (xy 170.18 154.94) (xy 170.18 165.68642)))
+    (feature2 (pts (xy 116.84 154.94) (xy 116.84 165.68642)))
+    (crossbar (pts (xy 116.84 165.099999) (xy 170.18 165.099999)))
+    (arrow1a (pts (xy 170.18 165.099999) (xy 169.053496 165.68642)))
+    (arrow1b (pts (xy 170.18 165.099999) (xy 169.053496 164.513578)))
+    (arrow2a (pts (xy 116.84 165.099999) (xy 117.966504 165.68642)))
+    (arrow2b (pts (xy 116.84 165.099999) (xy 117.966504 164.513578)))
+  )
+  (dimension 59.69 (width 0.15) (layer Dwgs.User)
+    (gr_text "59.690 mm" (at 105.380001 125.095 270) (layer Dwgs.User)
+      (effects (font (size 1 1) (thickness 0.15)))
+    )
+    (feature1 (pts (xy 116.84 154.94) (xy 106.09358 154.94)))
+    (feature2 (pts (xy 116.84 95.25) (xy 106.09358 95.25)))
+    (crossbar (pts (xy 106.680001 95.25) (xy 106.680001 154.94)))
+    (arrow1a (pts (xy 106.680001 154.94) (xy 106.09358 153.813496)))
+    (arrow1b (pts (xy 106.680001 154.94) (xy 107.266422 153.813496)))
+    (arrow2a (pts (xy 106.680001 95.25) (xy 106.09358 96.376504)))
+    (arrow2b (pts (xy 106.680001 95.25) (xy 107.266422 96.376504)))
+  )
+  (dimension 92.71 (width 0.15) (layer Dwgs.User)
+    (gr_text "92.710 mm" (at 181.64 113.665 270) (layer Dwgs.User)
+      (effects (font (size 1 1) (thickness 0.15)))
+    )
+    (feature1 (pts (xy 175.26 160.02) (xy 180.926421 160.02)))
+    (feature2 (pts (xy 175.26 67.31) (xy 180.926421 67.31)))
+    (crossbar (pts (xy 180.34 67.31) (xy 180.34 160.02)))
+    (arrow1a (pts (xy 180.34 160.02) (xy 179.753579 158.893496)))
+    (arrow1b (pts (xy 180.34 160.02) (xy 180.926421 158.893496)))
+    (arrow2a (pts (xy 180.34 67.31) (xy 179.753579 68.436504)))
+    (arrow2b (pts (xy 180.34 67.31) (xy 180.926421 68.436504)))
+  )
+  (dimension 63.5 (width 0.15) (layer Dwgs.User)
+    (gr_text "63.500 mm" (at 143.51 60.93) (layer Dwgs.User)
+      (effects (font (size 1 1) (thickness 0.15)))
+    )
+    (feature1 (pts (xy 175.26 67.31) (xy 175.26 61.643579)))
+    (feature2 (pts (xy 111.76 67.31) (xy 111.76 61.643579)))
+    (crossbar (pts (xy 111.76 62.23) (xy 175.26 62.23)))
+    (arrow1a (pts (xy 175.26 62.23) (xy 174.133496 62.816421)))
+    (arrow1b (pts (xy 175.26 62.23) (xy 174.133496 61.643579)))
+    (arrow2a (pts (xy 111.76 62.23) (xy 112.886504 62.816421)))
+    (arrow2b (pts (xy 111.76 62.23) (xy 112.886504 61.643579)))
+  )
   (gr_text "-  +" (at 142.24 93.98) (layer F.SilkS)
     (effects (font (size 1 1) (thickness 0.15)))
   )
-  (gr_line (start 175.26 68.58) (end 111.76 68.58) (layer Edge.Cuts) (width 0.05))
-  (gr_line (start 175.26 160.02) (end 175.26 68.58) (layer Edge.Cuts) (width 0.05))
+  (gr_line (start 175.26 67.31) (end 111.76 67.31) (layer Edge.Cuts) (width 0.05))
+  (gr_line (start 175.26 160.02) (end 175.26 67.31) (layer Edge.Cuts) (width 0.05))
   (gr_line (start 111.76 160.02) (end 175.26 160.02) (layer Edge.Cuts) (width 0.05))
-  (gr_line (start 111.76 68.58) (end 111.76 160.02) (layer Edge.Cuts) (width 0.05))
+  (gr_line (start 111.76 67.31) (end 111.76 160.02) (layer Edge.Cuts) (width 0.05))
   (segment (start 167.64 123.36) (end 167.64 124.46) (width 0.25) (layer B.Cu) (net 3))
   (segment (start 163.66 119.38) (end 167.64 123.36) (width 0.25) (layer B.Cu) (net 3))
@@
     (polygon
       (pts
-        (xy 111.76 68.58) (xy 175.26 68.58) (xy 175.26 160.02) (xy 111.76 160.02)
+        (xy 111.76 67.31) (xy 175.26 67.31) (xy 175.26 160.02) (xy 111.76 160.02)
       )
     )
@@
     (polygon
       (pts
-        (xy 111.76 68.58) (xy 175.26 68.58) (xy 175.26 160.02) (xy 111.76 160.02)
+        (xy 111.76 67.31) (xy 175.26 67.31) (xy 175.26 160.02) (xy 111.76 160.02)
       )
     )
